File: Hardware/MotorDriverPCB/evenFieldDriverBoard.brd (EAGLE design)
At the start: 86.3 x 36.5 mm, 17 parts, among them IC1 555, IC2 7805TV, J1 1X2-3.5MM

Commit message: Added build notes and BOM for motor driver board.
Parts:
- renumbered JP1 to HBRIDGEOUT, U$1 to HBRIDGEIN
Connections:
- net N$1 renamed VIN
Changed lines of the file:
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@@
 <element name="IC2" library="linear" library_urn="urn:adsk.eagle:library:262" package="TO220V" package3d_urn="urn:adsk.eagle:package:16417/1" value="7805TV" x="83.82" y="27.94"/>
 <element name="J1" library="adafruit" library_urn="urn:adsk.eagle:library:420" package="1X2-3.5MM" value="1X2-3.5MM" x="148.59" y="29.21" rot="R90"/>
-<element name="JP1" library="adafruit" library_urn="urn:adsk.eagle:library:420" package="1X06" value="" x="139.7" y="34.29" rot="R270"/>
+<element name="HBRIDGEOUT" library="adafruit" library_urn="urn:adsk.eagle:library:420" package="1X06" value="" x="139.7" y="34.29" rot="R270"/>
 <element name="R1" library="resistor" library_urn="urn:adsk.eagle:library:348" package="0309V" package3d_urn="urn:adsk.eagle:package:26090/1" value="10k" x="95.25" y="38.1" rot="R180"/>
 <element name="R2" library="pot" library_urn="urn:adsk.eagle:library:331" package="RJ9W" package3d_urn="urn:adsk.eagle:package:22702/1" value="100k" x="114.3" y="40.64" rot="R90"/>
-<element name="U$1" library="adafruit" library_urn="urn:adsk.eagle:library:420" package="1X10-BIG" value="PINHD-1X10" x="124.46" y="34.29" rot="R90"/>
+<element name="HBRIDGEIN" library="adafruit" library_urn="urn:adsk.eagle:library:420" package="1X10-BIG" value="PINHD-1X10" x="124.46" y="34.29" rot="R90"/>
 <element name="JP2" library="adafruit" library_urn="urn:adsk.eagle:library:420" package="1X01" value="" x="71.12" y="17.78"/>
 <element name="JP3" library="adafruit" library_urn="urn:adsk.eagle:library:420" package="1X01" value="" x="71.12" y="15.24"/>
@@
 <contactref element="R1" pad="2"/>
 <contactref element="IC1" pad="4"/>
-<contactref element="U$1" pad="3"/>
-<contactref element="U$1" pad="9"/>
+<contactref element="HBRIDGEIN" pad="3"/>
+<contactref element="HBRIDGEIN" pad="9"/>
 <wire x1="86.36" y1="25.4" x2="86.36" y2="30.48" width="1.27" layer="16"/>
 <wire x1="86.36" y1="30.48" x2="86.36" y2="33.02" width="1.27" layer="16"/>
@@
 <wire x1="93.98" y1="33.02" x2="101.6" y2="25.4" width="1.27" layer="16"/>
 <wire x1="93.98" y1="38.1" x2="93.98" y2="33.02" width="1.27" layer="16"/>
-<contactref element="U$1" pad="4"/>
+<contactref element="HBRIDGEIN" pad="4"/>
 <wire x1="124.46" y1="27.94" x2="124.46" y2="30.48" width="1.27" layer="16"/>
 <wire x1="124.46" y1="43.18" x2="127" y2="43.18" width="1.27" layer="16"/>
@@
 <contactref element="IC2" pad="1"/>
 <contactref element="C4" pad="+"/>
-<contactref element="U$1" pad="10"/>
+<contactref element="HBRIDGEIN" pad="10"/>
 <contactref element="S1" pad="2"/>
 <wire x1="81.28" y1="17.78" x2="81.28" y2="25.4" width="1.27" layer="16"/>
@@
 <contactref element="C1" pad="-"/>
 <contactref element="C2" pad="2"/>
-<contactref element="U$1" pad="2"/>
-<contactref element="U$1" pad="8"/>
+<contactref element="HBRIDGEIN" pad="2"/>
+<contactref element="HBRIDGEIN" pad="8"/>
 <contactref element="JP3" pad="1"/>
 <wire x1="83.82" y1="25.4" x2="83.82" y2="30.48" width="1.27" layer="16"/>
@@
 </signal>
 <signal name="N$11">
-<contactref element="U$1" pad="1"/>
+<contactref element="HBRIDGEIN" pad="1"/>
 <contactref element="IC1" pad="3"/>
 <wire x1="99.06" y1="25.4" x2="99.06" y2="22.86" width="1.27" layer="16"/>
@@
 </signal>
 <signal name="N$16">
-<contactref element="JP1" pad="5"/>
+<contactref element="HBRIDGEOUT" pad="5"/>
 <contactref element="J1" pad="1"/>
 <wire x1="139.7" y1="30.48" x2="148.59" y2="31.01" width="1.27" layer="1"/>
 </signal>
 <signal name="N$17">
-<contactref element="JP1" pad="6"/>
+<contactref element="HBRIDGEOUT" pad="6"/>
 <contactref element="J1" pad="2"/>
 <wire x1="148.59" y1="27.51" x2="139.7" y2="27.94" width="1.27" layer="1"/>
 </signal>
-<signal name="N$1">
+<signal name="VIN">
 <contactref element="JP2" pad="1"/>
 <contactref element="S1" pad="3"/>
