File: Hardware/MotorDriverPCB/evenFieldDriverBoard.sch (EAGLE design)
At the start: 17 parts, among them IC1 555, IC2 7805TV, J1 1X2-3.5MM

Commit message: Added build notes and BOM for motor driver board.
Parts:
- renumbered JP1 to HBRIDGEOUT, U$1 to HBRIDGEIN
Connections:
- net N$1 renamed VIN
